File: Hardware/Radio Knobs.kicad_sch (KiCad schematic)
At the start: 29 parts, among them J1 Conn_01x02, J2 Conn_01x02, J3 Conn_02x05_Odd_Even, SW2 N/A, SW4 Self-Return Rotary Switch

Commit message: Some progress made. Maybe one day I'll finish this...
Parts:
- removed D4: 15V, symbol Device:D_Zener
- removed R4: 100kΩ, symbol Device:R_Small
- added C5, C6: 1μF, symbol Device:C_Small
- added D4: LED, symbol Device:LED
- added R10, R6, R7: 100kΩ, symbol Device:R_Small
- added R3: 10k, symbol Device:R_Small
- added U1: MIC5317-3.3, symbol .Radio Knobs:MIC5317-3.3YM5
- C1: Comments (none) -> C1 has to be rated for the Zener Voltage of D2
- D1, D3: Comments (none) -> Zener 15V, 250mW, ±5%, SOT23; Digikey PN (none) -> 1727-2127-1-ND; MPN (none) -> BZX84-C15,235; Manufacturer (none) -> Nexperia
- D2: now not fitted
- R5: value 300kΩ -> 100kΩ
- renumbered R3 to R4, R13 to R8, R12 to R9
Connections:
- net +3V3: now also C4.1, R8.1, C6.1, R10.1, U1.5 (VOUT)
- net GND: now also C5.2, C6.2, D4.1 (K), U1.2 (GND)
- net VIN: now also R3.1; no longer D2.1 (K)
- net VOUT: now also C5.1, U1.1 (VIN), U1.3 (EN); no longer C4.1, R8.1
- net VA: now reaches C1.2, C2.2, D2.2 (A), D3.2 (A), R2.2, R4.2
- net VA: now also Q1.7 (D), Q1.8 (D)
- net at D1.2 (A), R8.2, R9.1: now also R7.1; no longer R5.2
- net at C4.2, Q1.2 (G): now also R5.2; no longer R5.1
- new net: D2.1 (K), R3.2
- new net: R5.1, R6.1
- new net: D4.2 (A), R10.2
- new net: R6.2, R7.2
- no-connect marks 2 -> 5
Other:
- note added: "(Three in series because I have lots of these already)"
- note added: "5.5mm Barrel connector"
- note added: "A solder bridge to select if the system will power on automatically when we have VIN, or if we still need to flick the switch"
- note added: "An LED to signal power would be connected to 20V. Even @5mA, that's 100mW wasted, which seems a lot. The "Raspberry Powered" is more useful, I think and can be connected to 3V3"
- note added: "Auto-On"
- note added: "Headers"
- note added: "Power Flags, misc..."
- note added: "Power LED"
- note added: "Rotary Encoder - Volume"
- note added: "Self Rerturn Rotary - Power"
- note added: "Switches"
- note added: "The Circuit"
- note added: "Zener Bias is 1mA@15V For a Vin of 20V -> Rzener = 5/1m = 5kΩ Zener Dissipation = 15mW As we already use 10kΩ, use that (halves dissipation)"
- moved on the sheet: C1, C4, C6, C7, D1, J1, J2, J3, JP1, Q1A, R14, R15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
